Commit message: Modified DAE scale down to 0.001

File: da_lamp_description/da_lamp_v2.urdf (robot description, URDF)
Before this commit: robot da_lamp_v2, 10 links, 9 joints
Joints:
- joint Rev11: axis 0.004434 -0.008963 0.0 -> 0.0 0.01 0.0; origin xyz=-0.017443 0.052175 -0.0075 rpy=0 0 0 -> xyz=0.0075 0.052175 -0.0075 rpy=0 0 0

Commit message: Added mimic joint for parallel robot

File: da_lamp_description/da_lamp_v2.urdf (robot description, URDF)
Before this commit: robot da_lamp_v2, 10 links, 9 joints
Joints:
- joint Rev3: mimic (none) -> joint=Rev2 multiplier=1 offset=0
- joint Rev4: mimic (none) -> joint=Rev2 multiplier=1 offset=0
- joint Rev7: mimic (none) -> joint=Rev6 multiplier=1 offset=0
- joint Rev8: mimic (none) -> joint=Rev6 multiplier=1 offset=0
